Commit message: feat(go2_ws): Add the xt16 lidar link in the Go2 URDF model.
Set the argument `enable_xt16` to `True` if you want to use lidar.

Note that the transform from lidar base to lidar frame is computed from hesai_description, since we use `imu_link` as parent, we need to invert the transform in our URDF model. The transform from Go2 to lidar is copied from the Unitree docs.

Reference:
- https://github.com/ori-drs/hesai_description/blob/834ed126aef58bba51853c6fe900c808c5f6310a/urdf/hesai_xt32.urdf.xacro#L38-L40
- https://support.unitree.com/home/en/developer/SLAM%20and%20Navigation_service

File: go2_ws/src/go2_description/xacro/robot.xacro (robot description, xacro)
@@ -4,6 +4,8 @@
     <!-- Declare argument -->
     <xacro:arg name="enable_gazebo" default="False"/>
+    <xacro:arg name="enable_xt16" default="False"/>
     <!-- Declare parameters -->
     <xacro:property name="enable_gazebo" value="$(arg enable_gazebo)"/>
+    <xacro:property name="enable_xt16" value="$(arg enable_xt16)"/>
     <!-- Include other file -->
     <xacro:include filename="$(find go2_description)/xacro/const.xacro"/>
@@ -113,3 +115,20 @@
         <axis xyz="0 0 0" />
     </joint>
+    <!-- xt16 lidar -->
+    <xacro:if value="${enable_xt16}">
+        <link name="xt16_link">
+            <visual>
+                <origin xyz="0 0 -0.0464" rpy="0 0 -1.5708" />
+                <geometry>
+                    <mesh filename="package://go2_description/dae/xt32.dae" scale="1 1 1"/>
+                </geometry>
+            </visual>
+        </link>
+        <joint name="xt16_lidar_mount_joint" type="fixed">
+            <origin xyz="0.171 0 0.0908" rpy="0 0 1.5708" />
+            <parent link="imu_link" />
+            <child link="xt16_link" />
+            <axis xyz="0 0 0" />
+        </joint>
+    </xacro:if>
 </robot>

Commit message: feat(go2_ws): Add the realsense link in the Go2 URDF model.
Because the Unitree does not provide the transform of the Realsense position, the current `realsense_mount_link` position is measured from the actual machine, and the `realsense_link` to `realsense_mount_link` is referenced from the unofficial Go2 SDK repo.

Reference:
- https://github.com/IntelRealSense/realsense-ros/tree/1cbd81be81e807eefb46f098e76381888ffc7001
- https://github.com/abizovnuralem/go2_ros2_sdk/blob/c9812a19b1116326760f2468bd9d6e228c635f81/go2_robot_sdk/urdf/go2_with_realsense.urdf#L1279-L1349

File: go2_ws/src/go2_description/xacro/robot.xacro (robot description, xacro)
@@ -5,7 +5,9 @@
     <xacro:arg name="enable_gazebo" default="False"/>
     <xacro:arg name="enable_xt16" default="False"/>
+    <xacro:arg name="enable_realsense" default="False"/>
     <!-- Declare parameters -->
     <xacro:property name="enable_gazebo" value="$(arg enable_gazebo)"/>
     <xacro:property name="enable_xt16" value="$(arg enable_xt16)"/>
+    <xacro:property name="enable_realsense" value="$(arg enable_realsense)"/>
     <!-- Include other file -->
     <xacro:include filename="$(find go2_description)/xacro/const.xacro"/>
@@ -132,3 +134,45 @@
         </joint>
     </xacro:if>
+    <!-- Realsense D435i camera -->
+    <!-- If you want to adjust the angle of realsense up or down,
+         please modify the rpy values in the `realsense_joint`. -->
+    <xacro:if value="${enable_realsense}">
+        <!-- camera mount link -->
+        <link name="realsense_mount_link"/>
+        <joint name="realsense_mount_joint" type="fixed">
+            <origin xyz="0.035 0 0.072" rpy="0 0 0" />
+            <parent link="Head_upper" />
+            <child link="realsense_mount_link" />
+            <axis xyz="0 0 0" />
+        </joint>
+        <!-- camera link -->
+        <link name="realsense_link">
+            <inertial>
+                <origin xyz="0 0 0" rpy="0 0 0" />
+                <mass value="0.072" />
+                <inertia ixx="0.0000215" ixy="0" ixz="0" iyy="0.0000302" iyz="0" izz="0.0000330" />
+            </inertial>
+            <visual>
+                <origin xyz="0.02 0 0" rpy="-1.5708 3.14 -1.5708 " />
+                <geometry>
+                    <mesh filename="package://realsense2_description/meshes/d435.dae" scale="1 1 1"/>
+                </geometry>
+                <material name="dark_grey">
+                    <color rgba="0.1 0.1 0.1 1" />
+                </material>
+            </visual>
+            <collision>
+                <origin xyz="0.01 0 0" rpy="0 0 0" />
+                <geometry>
+                    <box size="0.025 0.09 0.025" />
+                </geometry>
+            </collision>
+        </link>
+        <joint name="realsense_joint" type="fixed">
+            <origin xyz="0 0 0" rpy="0 0 0" />
+            <parent link="realsense_mount_link" />
+            <child link="realsense_link" />
+            <axis xyz="0 0 0" />
+        </joint>
+    </xacro:if>
 </robot>
